Commit message: urdf: make robot move in gazebo

File: src/urdf_test/description/gazebo_control.xacro (robot description, xacro)
@@ -9,4 +9,10 @@
             <wheel_separation>0.35</wheel_separation>
             <wheel_diameter>${wheel_link_diameter}</wheel_diameter>
+            <topic>cmd_vel</topic>
+            <tf_topic>tf</tf_topic>
+            <odom_topic>odom</odom_topic>
+            <frame_id>odom</frame_id>
+            <child_frame_id>base_link</child_frame_id>
+            <odom_publisher_frequency>30</odom_publisher_frequency>
             <!-- Limits -->
             <max_wheel_torque>200</max_wheel_torque>
@@ -17,5 +23,5 @@
             <publish_odom>true</publish_odom>
             <publish_odom_tf>true</publish_odom_tf>
-            <publish_wheel_tf>true</publish_wheel_tf>
+            <publish_wheel_tf>false</publish_wheel_tf>
         </plugin>
         <!-- Joint state publisher -->

File: src/urdf_test/description/model.urdf.xacro (robot description, xacro)
@@ -63,9 +63,9 @@
     <joint name="right_wheel_joint" type="continuous">
         <parent link="base_link"/>
-        <child link="right_wheel"/>
+        <child link="right_wheel_link"/>
         <origin xyz="0 -${chassis_link_y/2} ${wheel_link_diameter/2}" rpy="${pi/2} 0 0" />
         <axis xyz="0 0 -1"/>
     </joint>
-    <link name="right_wheel">
+    <link name="right_wheel_link">
         <visual>
             <geometry>
