Commit message: urdf_test: switch mecanum controller to ros2_control

File: src/urdf_test/description/gazebo_control.xacro (robot description, xacro)
@@ -2,29 +2,23 @@
 <robot xmlns:xacro="http://www.ros.org/wiki/xacro">
     <xacro:include filename="$(find urdf_test)/description/constants.xacro" />
+    <ros2_control name="GazeboSimSystem" type="system">
+        <hardware>
+            <plugin>gz_ros2_control/GazeboSimSystem</plugin>
+        </hardware>
+        <xacro:macro name="wheel_iface" params="name">
+            <joint name="${name}_wheel_joint">
+                <command_interface name="velocity"/>
+                <state_interface name="position"/>
+                <state_interface name="velocity"/>
+            </joint>
+        </xacro:macro>
+        <xacro:wheel_iface name="front_left"/>
+        <xacro:wheel_iface name="front_right"/>
+        <xacro:wheel_iface name="rear_left"/>
+        <xacro:wheel_iface name="rear_right"/>
+    </ros2_control>
     <gazebo>
-        <plugin filename="gz-sim-mecanum-drive-system" name="gz::sim::systems::MecanumDrive">
-            <!-- Wheel Information -->
-            <front_left_joint>front_left_wheel_joint</front_left_joint>
-            <front_right_joint>front_right_wheel_joint</front_right_joint>
-            <back_left_joint>rear_left_wheel_joint</back_left_joint>
-            <back_right_joint>rear_right_wheel_joint</back_right_joint>
-            <wheelbase>${wheel_base_x}</wheelbase>
-            <wheel_separation>${wheel_track_y}</wheel_separation>
-            <wheel_radius>${wheel_link_diameter/2}</wheel_radius>
-            <topic>cmd_vel</topic>
-            <tf_topic>tf</tf_topic>
-            <odom_topic>odom</odom_topic>
-            <frame_id>odom</frame_id>
-            <child_frame_id>base_link</child_frame_id>
-            <odom_publisher_frequency>30</odom_publisher_frequency>
-        </plugin>
-        <!-- Joint state publisher -->
-        <plugin filename="gz-sim-joint-state-publisher-system"
-            name="gz::sim::systems::JointStatePublisher">
-            <topic>joint_states</topic>
-            <joint_name>front_left_wheel_joint</joint_name>
-            <joint_name>front_right_wheel_joint</joint_name>
-            <joint_name>rear_left_wheel_joint</joint_name>
-            <joint_name>rear_right_wheel_joint</joint_name>
+        <plugin filename="gz_ros2_control-system" name="gz_ros2_control::GazeboSimROS2ControlPlugin">
+            <parameters>$(find urdf_test)/config/controllers.yaml</parameters>
         </plugin>
     </gazebo>
