Commit message: urdf_test: fix aruco orientation

File: src/urdf_test/description/aruco.xacro (robot description, xacro)
@@ -28,5 +28,5 @@
         <parent link="base_link"/>
         <child link="aruco_link"/>
-        <origin xyz="0 0 0.1" rpy="0 0 1.57"/>
+        <origin xyz="0 0 0.1" rpy="0 0 ${-pi}"/>
     </joint>
 </robot>
