Commit message: urdf_test: switch model to mecanum 27

File: src/urdf_test/description/constants.xacro (robot description, xacro)
@@ -1,8 +1,18 @@
 <?xml version="1.0"?>
 <robot xmlns:xacro="http://www.ros.org/wiki/xacro">
-    <xacro:property name="chassis_link_x" value="0.1" />
-    <xacro:property name="chassis_link_y" value="0.07" />
-    <xacro:property name="chassis_link_z" value="0.06" />
-    <xacro:property name="wheel_link_diameter" value="0.05" />
-    <xacro:property name="wheel_link_length" value="0.01" />
+    <xacro:property name="chassis_link_x" value="0.250" />
+    <xacro:property name="chassis_link_y" value="0.167" />
+    <xacro:property name="chassis_link_z" value="0.082" />
+    <!-- Mecanum wheels, 104 mm diameter, 38 mm wide -->
+    <xacro:property name="wheel_link_diameter" value="0.104" />
+    <xacro:property name="wheel_link_length" value="0.038" />
+    <!-- Distance between wheel centers, 216 mm (x, wheelbase) by 168 mm (y, track) -->
+    <xacro:property name="wheel_base_x" value="0.216" />
+    <xacro:property name="wheel_track_y" value="0.168" />
+    <!-- Axle height above the ground (wheels touch the ground).
+         The axle sits at the chassis mid-height, so the chassis center is at this same height. -->
+    <xacro:property name="wheel_axle_z" value="${wheel_link_diameter/2}" />
+    <xacro:property name="chassis_center_z" value="${wheel_axle_z}" />
+    <xacro:property name="chassis_mass" value="0.5" />
+    <xacro:property name="wheel_mass" value="0.1" />
 </robot>

File: src/urdf_test/description/gazebo_control.xacro (robot description, xacro)
@@ -3,9 +3,12 @@
     <xacro:include filename="$(find urdf_test)/description/constants.xacro" />
     <gazebo>
-        <plugin filename="gz-sim-diff-drive-system" name="gz::sim::systems::DiffDrive">
+        <plugin filename="gz-sim-mecanum-drive-system" name="gz::sim::systems::MecanumDrive">
             <!-- Wheel Information -->
-            <left_joint>left_wheel_joint</left_joint>
-            <right_joint>right_wheel_joint</right_joint>
-            <wheel_separation>${chassis_link_y+wheel_link_length*2}</wheel_separation>
+            <front_left_joint>front_left_wheel_joint</front_left_joint>
+            <front_right_joint>front_right_wheel_joint</front_right_joint>
+            <back_left_joint>rear_left_wheel_joint</back_left_joint>
+            <back_right_joint>rear_right_wheel_joint</back_right_joint>
+            <wheelbase>${wheel_base_x}</wheelbase>
+            <wheel_separation>${wheel_track_y}</wheel_separation>
             <wheel_radius>${wheel_link_diameter/2}</wheel_radius>
             <topic>cmd_vel</topic>
@@ -15,13 +18,4 @@
             <child_frame_id>base_link</child_frame_id>
             <odom_publisher_frequency>30</odom_publisher_frequency>
-            <!-- Limits -->
-            <max_wheel_torque>200</max_wheel_torque>
-            <max_wheel_acceleration>10.0</max_wheel_acceleration>
-            <!-- Output -->
-            <odometry_frame>odom</odometry_frame>
-            <robot_base_frame>base_link</robot_base_frame>
-            <publish_odom>true</publish_odom>
-            <publish_odom_tf>true</publish_odom_tf>
-            <publish_wheel_tf>false</publish_wheel_tf>
         </plugin>
         <!-- Joint state publisher -->
@@ -29,6 +23,8 @@
             name="gz::sim::systems::JointStatePublisher">
             <topic>joint_states</topic>
-            <joint_name>left_wheel_joint</joint_name>
-            <joint_name>right_wheel_joint</joint_name>
+            <joint_name>front_left_wheel_joint</joint_name>
+            <joint_name>front_right_wheel_joint</joint_name>
+            <joint_name>rear_left_wheel_joint</joint_name>
+            <joint_name>rear_right_wheel_joint</joint_name>
         </plugin>
     </gazebo>

File: src/urdf_test/description/model.urdf.xacro (robot description, xacro)
@@ -1,4 +1,4 @@
 <?xml version="1.0"?>
-<robot xmlns:xacro="http://www.ros.org/wiki/xacro" name="robot">
+<robot xmlns:xacro="http://www.ros.org/wiki/xacro" xmlns:gz="http://gazebosim.org/schema" name="robot">
     <xacro:include filename="$(find urdf_test)/description/constants.xacro" />
     <xacro:include filename="$(find urdf_test)/description/inertia.xacro" />
@@ -7,8 +7,9 @@
     <xacro:include filename="$(find urdf_test)/description/aruco.xacro" />
     <link name="base_link"></link>
-    <!-- Chassis link -->
+    <!-- Chassis link (250 x 167 x 82 mm), centered at wheel axle height -->
     <joint name="chassis_joint" type="fixed">
         <parent link="base_link"/>
         <child link="chassis_link"/>
+        <origin xyz="0 0 ${chassis_center_z}" rpy="0 0 0"/>
     </joint>
     <link name="chassis_link">
@@ -17,5 +18,4 @@
                 <box size="${chassis_link_x} ${chassis_link_y} ${chassis_link_z}" />
             </geometry>
-            <origin xyz="${chassis_link_x/3} 0 ${chassis_link_z/2 + wheel_link_diameter/3}" rpy="0 0 0"/>
             <material name="blue" />
         </visual>
@@ -24,8 +24,7 @@
                 <box size="${chassis_link_x} ${chassis_link_y} ${chassis_link_z}" />
             </geometry>
-            <origin xyz="${chassis_link_x/3} 0 ${chassis_link_z/2 + wheel_link_diameter/3}" rpy="0 0 0"/>
         </collision>
-        <xacro:inertial_box mass="0.5" x="${chassis_link_x}" y="${chassis_link_y}" z="${chassis_link_x}">
-            <origin xyz="${chassis_link_x/3} 0 ${chassis_link_z/2 + wheel_link_diameter/3}" rpy="0 0 0"/>
+        <xacro:inertial_box mass="${chassis_mass}" x="${chassis_link_x}" y="${chassis_link_y}" z="${chassis_link_z}">
+            <origin xyz="0 0 0" rpy="0 0 0"/>
         </xacro:inertial_box>
     </link>
@@ -33,86 +32,45 @@
         <material>Gazebo/Blue</material>
     </gazebo>
-    <!-- Left wheel link -->
-    <joint name="left_wheel_joint" type="continuous">
-        <parent link="base_link"/>
-        <child link="left_wheel_link"/>
-        <origin xyz="0 ${chassis_link_y/2} ${wheel_link_diameter/2}" rpy="-${pi/2} 0 0" />
-        <axis xyz="0 0 1"/>
-    </joint>
-    <link name="left_wheel_link">
-        <visual>
-            <geometry>
-                <cylinder radius="${wheel_link_diameter/2}" length="${wheel_link_length}"/>
-            </geometry>
-            <origin xyz="0 0 ${wheel_link_length/2}"/>
-            <material name="orange"/>
-        </visual>
-        <collision>
-            <geometry>
-                <cylinder radius="${wheel_link_diameter/2}" length="${wheel_link_length}"/>
-            </geometry>
-            <origin xyz="0 0 ${wheel_link_length/2}"/>
-        </collision>
-        <xacro:inertial_cylinder mass="0.1" length="${wheel_link_length}" radius="${wheel_link_diameter/2}">
-            <origin xyz="0 0 ${wheel_link_length/2}" />
-        </xacro:inertial_cylinder>
-    </link>
-    <gazebo reference="left_wheel_link">
-        <material>Gazebo/Orange</material>
-    </gazebo>
-    <!-- Right wheel link -->
-    <joint name="right_wheel_joint" type="continuous">
-        <parent link="base_link"/>
-        <child link="right_wheel_link"/>
-        <origin xyz="0 -${chassis_link_y/2} ${wheel_link_diameter/2}" rpy="${pi/2} 0 0" />
-        <axis xyz="0 0 -1"/>
-    </joint>
-    <link name="right_wheel_link">
-        <visual>
-            <geometry>
-                <cylinder radius="${wheel_link_diameter/2}" length="${wheel_link_length}"/>
-            </geometry>
-            <origin xyz="0 0 ${wheel_link_length/2}"/>
-            <material name="orange"/>
-        </visual>
-        <collision>
-            <geometry>
-                <cylinder radius="${wheel_link_diameter/2}" length="${wheel_link_length}"/>
-            </geometry>
-            <origin xyz="0 0 ${wheel_link_length/2}"/>
-        </collision>
-        <xacro:inertial_cylinder mass="0.1" length="${wheel_link_length}" radius="${wheel_link_diameter/2}">
-            <origin xyz="0 0 ${wheel_link_length/2}" />
-        </xacro:inertial_cylinder>
-    </link>
-    <gazebo reference="right_wheel_link">
-        <material>Gazebo/Orange</material>
-    </gazebo>
-    <!-- Caster wheel link -->
-        <joint name="caster_joint" type="fixed">
-        <parent link="base_link"/>
-        <child link="caster_link"/>
-        <origin xyz="${chassis_link_x/2} 0 ${wheel_link_diameter/2}"/>
-    </joint>
-    <link name="caster_link">
-        <visual>
-            <geometry>
-                <sphere radius="${wheel_link_diameter/2}"/>
-            </geometry>
-            <material name="orange"/>
-        </visual>
-        <collision>
-            <geometry>
-                <sphere radius="${wheel_link_diameter/2}"/>
-            </geometry>
-        </collision>
-        <xacro:inertial_sphere mass="0.1" radius="0.05">
-            <origin xyz="0 0 0" rpy="0 0 0"/>
-        </xacro:inertial_sphere>
-    </link>
-    <gazebo reference="caster_link">
-        <material>Gazebo/Orange</material>
-        <mu1 value="0.001"/>
-        <mu2 value="0.001"/>
-    </gazebo>
+    <xacro:macro name="mecanum_wheel" params="prefix x y fdir">
+        <joint name="${prefix}_wheel_joint" type="continuous">
+            <parent link="base_link"/>
+            <child link="${prefix}_wheel_link"/>
+            <origin xyz="${x} ${y} ${wheel_axle_z}" rpy="${-pi/2} 0 0" />
+            <axis xyz="0 0 1"/>
+        </joint>
+        <link name="${prefix}_wheel_link">
+            <visual>
+                <geometry>
+                    <cylinder radius="${wheel_link_diameter/2}" length="${wheel_link_length}"/>
+                </geometry>
+                <material name="orange"/>
+            </visual>
+            <collision>
+                <geometry>
+                    <sphere radius="${wheel_link_diameter/2}"/>
+                </geometry>
+            </collision>
+            <xacro:inertial_cylinder mass="${wheel_mass}" length="${wheel_link_length}" radius="${wheel_link_diameter/2}">
+                <origin xyz="0 0 0" rpy="0 0 0" />
+            </xacro:inertial_cylinder>
+        </link>
+        <gazebo reference="${prefix}_wheel_link">
+            <material>Gazebo/Orange</material>
+            <collision>
+                <surface>
+                    <friction>
+                        <ode>
+                            <mu>1.0</mu>
+                            <mu2>0.0</mu2>
+                            <fdir1 gz:expressed_in="base_link">${fdir}</fdir1>
+                        </ode>
+                    </friction>
+                </surface>
+            </collision>
+        </gazebo>
+    </xacro:macro>
+    <xacro:mecanum_wheel prefix="front_left"  x="${ wheel_base_x/2}" y="${ wheel_track_y/2}" fdir="1 -1 0" />
+    <xacro:mecanum_wheel prefix="front_right" x="${ wheel_base_x/2}" y="${-wheel_track_y/2}" fdir="1 1 0" />
+    <xacro:mecanum_wheel prefix="rear_left"   x="${-wheel_base_x/2}" y="${ wheel_track_y/2}" fdir="1 1 0" />
+    <xacro:mecanum_wheel prefix="rear_right"  x="${-wheel_base_x/2}" y="${-wheel_track_y/2}" fdir="1 -1 0" />
 </robot>
